File: WiegandBoard/schematics/Wiegand.brd (EAGLE design)
At the start: 78.7 x 58.4 mm, 89 parts, among them J1 AVR_SPI_PRG_6NS, Q1 NTR1P02T1G, Q2 NTR1P02T1G, Q3 NTR1P02T1G, Q4 NTR1P02T1G, Q5 NTR1P02T1G, Q6 NTR1P02T1G, Q7 NTR1P02T1G, Q8 NTR1P02T1G, U1 ATMEGA168, U2 RS485_SP491, U4 MOC3063, U5 MOC3063, U6 MOC3063, U7 MOC3063, U8 MOC3063, U9 MOC3063, Y1 16Mhz

Commit message: REVC boards made
Parts:
- JP2: value First Node A -> (none)
- JP3: value Last Node Y -> (none)
- JP4: value First Node B -> (none)
- JP5: value Last Node Z -> (none)
- X4: device LumisenseV6:NOVA-LABS-LOGO-FULL-SMALL-2 -> NOVA-LABS-LOGO:NOVA-LABS-LOGO-SILK-400MIL
- moved X4 2.54 mm to (64.3, 22.6)
Other:
- board text added: "Rev C - 2014-02-28"
- board text removed: "Rev C - 2014-02-24"
