File: WiegandBoard/schematics/Wiegand.sch (EAGLE design)
At the start: 89 parts, among them IC1 MC33269ST-3.3T3, J1 AVR_SPI_PRG_6NS, Q1 NTR1P02T1G, Q2 NTR1P02T1G, Q3 NTR1P02T1G, Q4 NTR1P02T1G, Q5 NTR1P02T1G, Q6 NTR1P02T1G, Q7 NTR1P02T1G, Q8 NTR1P02T1G, U1 ATMEGA168, U2 RS485_SP491, U4 MOC3063, U5 MOC3063, U6 MOC3063, U7 MOC3063, U8 MOC3063, U9 MOC3063, Y1 16Mhz

Commit message: REVC boards made
Parts:
- JP2: value First Node A -> (none)
- JP3: value Last Node Y -> (none)
- JP4: value First Node B -> (none)
- JP5: value Last Node Z -> (none)
- LED10, LED11, LED12, LED13, LED14, LED15, LED16, LED2, LED3, LED5, LED6, LED7, LED8, LED9: MFG_PN LY R976-PS-36 -> LH R974-LP-1
- U4, U5, U6, U7, U8, U9: MFG_PN MOC3063M -> MOC3063S-TA1
- X4: device LumisenseV6:NOVA-LABS-LOGO-FULL-SMALL-2 -> NOVA-LABS-LOGO:NOVA-LABS-LOGO-SILK-400MIL
Other:
- note added: "FIRST NODE A"
- note added: "FIRST NODE B"
- note added: "LAST NODE Y"
- note added: "LAST NODE Z"
- note added: "Rev C - 2014-02-28"
- note removed: "Rev C - 2014-02-24"
Changed lines of the file:
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@@
 </part>
 <part name="LED2" library="dp_devices" deviceset="LED" device="-0805" value="RED">
-<attribute name="MFG_PN" value="LY R976-PS-36"/>
+<attribute name="MFG_PN" value="LH R974-LP-1"/>
 </part>
 <part name="LED3" library="dp_devices" deviceset="LED" device="-0805" value="RED">
-<attribute name="MFG_PN" value="LY R976-PS-36"/>
+<attribute name="MFG_PN" value="LH R974-LP-1"/>
 </part>
 <part name="R14" library="SparkFun" deviceset="RESISTOR" device="0603-RES" value="1K">
@@
 </part>
 <part name="GND14" library="SparkFun" deviceset="GND" device=""/>
-<part name="JP2" library="SparkFun" deviceset="JUMPER-2" device="PTH" value="First Node A">
+<part name="JP2" library="SparkFun" deviceset="JUMPER-2" device="PTH">
 <attribute name="MFG_PN" value="1x2 pin header"/>
 </part>
-<part name="JP3" library="SparkFun" deviceset="JUMPER-2" device="PTH" value="Last Node Y">
+<part name="JP3" library="SparkFun" deviceset="JUMPER-2" device="PTH">
 <attribute name="MFG_PN" value="1x2 pin header"/>
 </part>
-<part name="JP4" library="SparkFun" deviceset="JUMPER-2" device="PTH" value="First Node B">
+<part name="JP4" library="SparkFun" deviceset="JUMPER-2" device="PTH">
 <attribute name="MFG_PN" value="1x2 pin header"/>
 </part>
-<part name="JP5" library="SparkFun" deviceset="JUMPER-2" device="PTH" value="Last Node Z">
+<part name="JP5" library="SparkFun" deviceset="JUMPER-2" device="PTH">
 <attribute name="MFG_PN" value="1x2 pin header"/>
 </part>
@@
 </part>
 <part name="LED5" library="dp_devices" deviceset="LED" device="-0805" value="RED">
-<attribute name="MFG_PN" value="LY R976-PS-36"/>
+<attribute name="MFG_PN" value="LH R974-LP-1"/>
 </part>
 <part name="GND4" library="SparkFun" deviceset="GND" device=""/>
@@
 </part>
 <part name="LED6" library="dp_devices" deviceset="LED" device="-0805" value="RED">
-<attribute name="MFG_PN" value="LY R976-PS-36"/>
+<attribute name="MFG_PN" value="LH R974-LP-1"/>
 </part>
 <part name="GND7" library="SparkFun" deviceset="GND" device=""/>
@@
 </part>
 <part name="LED7" library="dp_devices" deviceset="LED" device="-0805" value="RED">
-<attribute name="MFG_PN" value="LY R976-PS-36"/>
+<attribute name="MFG_PN" value="LH R974-LP-1"/>
 </part>
 <part name="GND8" library="SparkFun" deviceset="GND" device=""/>
@@
 </part>
 <part name="LED8" library="dp_devices" deviceset="LED" device="-0805" value="RED">
-<attribute name="MFG_PN" value="LY R976-PS-36"/>
+<attribute name="MFG_PN" value="LH R974-LP-1"/>
 </part>
 <part name="GND15" library="SparkFun" deviceset="GND" device=""/>
@@
 </part>
 <part name="LED9" library="dp_devices" deviceset="LED" device="-0805" value="RED">
-<attribute name="MFG_PN" value="LY R976-PS-36"/>
+<attribute name="MFG_PN" value="LH R974-LP-1"/>
 </part>
 <part name="GND16" library="SparkFun" deviceset="GND" device=""/>
@@
 </part>
 <part name="LED10" library="dp_devices" deviceset="LED" device="-0805" value="RED">
-<attribute name="MFG_PN" value="LY R976-PS-36"/>
+<attribute name="MFG_PN" value="LH R974-LP-1"/>
 </part>
 <part name="GND17" library="SparkFun" deviceset="GND" device=""/>
@@
 <part name="GND18" library="SparkFun" deviceset="GND" device=""/>
 <part name="U4" library="SparkFun-DiscreteSemi" deviceset="MOC3063*" device="S" value="MOC3063">
-<attribute name="MFG_PN" value="MOC3063M"/>
+<attribute name="MFG_PN" value="MOC3063S-TA1"/>
 </part>
 <part name="P+18" library="SparkFun" deviceset="VCC" device=""/>
@@
 </part>
 <part name="LED11" library="dp_devices" deviceset="LED" device="-0805" value="RED">
-<attribute name="MFG_PN" value="LY R976-PS-36"/>
+<attribute name="MFG_PN" value="LH R974-LP-1"/>
 </part>
 <part name="U5" library="SparkFun-DiscreteSemi" deviceset="MOC3063*" device="S" value="MOC3063">
-<attribute name="MFG_PN" value="MOC3063M"/>
+<attribute name="MFG_PN" value="MOC3063S-TA1"/>
 </part>
 <part name="R11" library="SparkFun" deviceset="RESISTOR" device="0603-RES" value="440">
@@
 </part>
 <part name="LED12" library="dp_devices" deviceset="LED" device="-0805" value="RED">
-<attribute name="MFG_PN" value="LY R976-PS-36"/>
+<attribute name="MFG_PN" value="LH R974-LP-1"/>
 </part>
 <part name="U6" library="SparkFun-DiscreteSemi" deviceset="MOC3063*" device="S" value="MOC3063">
-<attribute name="MFG_PN" value="MOC3063M"/>
+<attribute name="MFG_PN" value="MOC3063S-TA1"/>
 </part>
 <part name="R12" library="SparkFun" deviceset="RESISTOR" device="0603-RES" value="440">
@@
 </part>
 <part name="LED13" library="dp_devices" deviceset="LED" device="-0805" value="RED">
-<attribute name="MFG_PN" value="LY R976-PS-36"/>
+<attribute name="MFG_PN" value="LH R974-LP-1"/>
 </part>
 <part name="U7" library="SparkFun-DiscreteSemi" deviceset="MOC3063*" device="S" value="MOC3063">
-<attribute name="MFG_PN" value="MOC3063M"/>
+<attribute name="MFG_PN" value="MOC3063S-TA1"/>
 </part>
 <part name="R19" library="SparkFun" deviceset="RESISTOR" device="0603-RES" value="440">
@@
 </part>
 <part name="LED14" library="dp_devices" deviceset="LED" device="-0805" value="RED">
-<attribute name="MFG_PN" value="LY R976-PS-36"/>
+<attribute name="MFG_PN" value="LH R974-LP-1"/>
 </part>
 <part name="U8" library="SparkFun-DiscreteSemi" deviceset="MOC3063*" device="S" value="MOC3063">
-<attribute name="MFG_PN" value="MOC3063M"/>
+<attribute name="MFG_PN" value="MOC3063S-TA1"/>
 </part>
 <part name="R20" library="SparkFun" deviceset="RESISTOR" device="0603-RES" value="440">
@@
 </part>
 <part name="LED15" library="dp_devices" deviceset="LED" device="-0805" value="RED">
-<attribute name="MFG_PN" value="LY R976-PS-36"/>
+<attribute name="MFG_PN" value="LH R974-LP-1"/>
 </part>
 <part name="U9" library="SparkFun-DiscreteSemi" deviceset="MOC3063*" device="S" value="MOC3063">
-<attribute name="MFG_PN" value="MOC3063M"/>
+<attribute name="MFG_PN" value="MOC3063S-TA1"/>
 </part>
 <part name="R21" library="SparkFun" deviceset="RESISTOR" device="0603-RES" value="440">
@@
 </part>
 <part name="LED16" library="dp_devices" deviceset="LED" device="-0805" value="RED">
-<attribute name="MFG_PN" value="LY R976-PS-36"/>
+<attribute name="MFG_PN" value="LH R974-LP-1"/>
 </part>
 <part name="LED17" library="dp_devices" deviceset="LED" device="-0805" value="YLW">
@@
 <attribute name="MFG_PN" value="NTR1P02T1G"/>
 </part>
-<part name="X4" library="LumisenseV6" deviceset="NOVA-LABS-LOGO" device="-FULL-SMALL-2"/>
+<part name="X4" library="NOVA-LABS-LOGO" deviceset="NOVA-LABS-LOGO" device="-SILK-400MIL"/>
 </parts>
 <sheets>
@@
 <text x="7.62" y="10.16" size="2.54" layer="94">Microcontroller</text>
 <text x="149.86" y="83.82" size="6.4516" layer="94">MakerPass - Wiegand Board</text>
-<text x="149.86" y="17.78" size="6.4516" layer="94">Rev C - 2014-02-24</text>
+<text x="149.86" y="17.78" size="6.4516" layer="94">Rev C - 2014-02-28</text>
 <text x="157.48" y="187.96" size="1.778" layer="91" rot="R180">FIRST NODE</text>
 <text x="203.2" y="187.96" size="1.778" layer="91" rot="R180">LAST NODE</text>
@@
 - Head-A --- Slave-Y
 - Head-B --- Slave-Z</text>
+<text x="152.4" y="172.72" size="1.27" layer="94" rot="R180">FIRST NODE A</text>
+<text x="152.4" y="149.86" size="1.27" layer="94" rot="R180">FIRST NODE B</text>
+<text x="190.5" y="147.32" size="1.27" layer="94">LAST NODE Z</text>
+<text x="190.5" y="170.18" size="1.27" layer="94">LAST NODE Y</text>
 </plain>
 <instances>
